File: ethernet.kicad_sch (KiCad schematic)
At the start: 57 parts, among them J1 L834-1G1T-S7, U20 KSZ9031RNXCA, Y2 Resonator_25MHz_ABM8G

Commit message: "In the process of upgrading the ddr memory"
Parts:
- R127, R148, R149, R150, R151, R152, R153, R155, R156, R157, R158, R159, R165, R166, R194: footprint antmicro-footprints:R_0402_1005Metric -> Resistor_SMD:R_0402_1005Metric
