File: interfaces.kicad_sch (KiCad schematic)
At the start: 135 parts, among them J3 USB-Micro-B_Amphenol_10118192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, J6 PinHeader_2x7_P2mm_Drill0.9mm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, J7 PinHeader_1x6_P2.54mm_Drill1.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, U1 SFEM016GB1ED1TO-I-5E-311-STD, U14 XC7A100T-FGG484, U17 USB3300-EZK-TR, U18 USB3300-EZK-TR, U19 FT4232H_QFN, U21 LSF0108RKSR, U22 LSF0101DRYR, U23 Oscillator_24MHz_ASEMB, U24 Oscillator_24MHz_ASEMB, U26 FT2232HQ, U27 93LCxxBxxOT, U6 NVT2008BQ,115, Y1 Resonator_12MHz_ABM8G

Commit message: "In the process of upgrading the ddr memory"
Parts:
- removed C10, C11, C12, C13, C18, C19, C20, C21, C22, C24, C248, C249, C25, C251, C252, C253, C254, C26, C4, C5: C_100n_0402, Capacitor_SMD:C_0402_1005Metric, symbol antmicroCapacitors0402:C_100n_0402
- removed C17, C39: C_100n_6V3_0402, Capacitor_SMD:C_0402_1005Metric, symbol antmicroCapacitorsmisc:C_100n_6V3_0402
- removed C177, C222, C23, C245, C246, C247: C_4u7_0402, Capacitor_SMD:C_0402_1005Metric, symbol antmicroCapacitors0402:C_4u7_0402
- removed J7: PinHeader_1x6_P2.54mm_Drill1.1mm, antmicro-footprints:PinHeader_1x6_P2.54mm_Drill1.1mm, symbol antmicroGenericPinHeaders:PinHeader_1x6_P2.54mm_Drill1.1mm
- removed R10, R11: R_0R_0402, antmicro-footprints:R_0402_1005Metric, symbol antmicroResistors0402:R_0R_0402
- removed R12, R53, R62: R_200k_0402, antmicro-footprints:R_0402_1005Metric, symbol antmicroResistors0402:R_200k_0402
- removed R45, R46, R47, R48, R49, R50, R51, R52: R_357k_0402, antmicro-footprints:R_0402_1005Metric, symbol antmicroResistors0402:R_357k_0402
- removed R5, R7: R_12k_0402, antmicro-footprints:R_0402_1005Metric, symbol antmicroResistors0402:R_12k_0402
- removed R6, R8: R_1k_0402, antmicro-footprints:R_0402_1005Metric, symbol antmicroResistors0402:R_1k_0402
- removed U17, U18: USB3300-EZK-TR, antmicro-footprints:QFN-32-1EP_5x5mm, symbol antmicroInterfaceControllers:USB3300-EZK-TR
- removed U19: FT4232H_QFN, antmicro-footprints:QFN-64-1EP_9x9mm_P0.5mm, symbol antmicroInterfaceControllers:FT4232H_QFN
- removed U21: LSF0108RKSR, antmicro-footprints:VQFN-20_1EP_4.5x2.5mm_P0.5mm, symbol antmicroLogicTranslatorsLevelShifters:LSF0108RKSR
- removed U22: LSF0101DRYR, antmicro-footprints:USON-6_1.45x1.0mm_P0.5mm_Texas_DRY6, symbol antmicroLogicTranslatorsLevelShifters:LSF0101DRYR
- removed U23, U24: Oscillator_24MHz_ASEMB, antmicro-footprints:Oscillator_SMD_Abracon_ASEMB_3.2x2.5mm, symbol antmicroOscillators:Oscillator_24MHz_ASEMB
- removed U6: NVT2008BQ,115, antmicro-footprints:VQFN-20_1EP_4.5x2.5mm_P0.5mm, symbol antmicroLogicTranslatorsLevelShifters:NVT2008BQ,115
- added H1: MountingHole, MountingHole:MountingHole_2.2mm_M2, symbol Mechanical:MountingHole
- added J2: Bus_M.2_Socket_M, artix-dc-scm:MDT275M02001, symbol Connector:Bus_M.2_Socket_M
- R117, R118, R119, R120, R121, R122, R123, R124, R125, R126, R143, R160, R191, R192, R193, R195, R196, R3, R9: footprint antmicro-footprints:R_0402_1005Metric -> Resistor_SMD:R_0402_1005Metric
Connections:
- new net: J2.1 (GND), J2.15 (GND), J2.21 (GND), J2.27 (GND), J2.3 (GND), J2.33 (GND), J2.39 (GND), J2.45 (GND), J2.51 (GND), J2.57 (GND), J2.71 (GND), J2.73 (GND), J2.75 (GND), J2.9 (GND)
- new net: J2.12 (3.3V), J2.14 (3.3V), J2.16 (3.3V), J2.18 (3.3V), J2.2 (3.3V), J2.4 (3.3V), J2.70 (3.3V), J2.72 (3.3V), J2.74 (3.3V)
- no-connect marks 105 -> 45
Other:
- note removed: "Debug USB"
- note removed: "ESPI level translation"
- note removed: "HPM SPI"
- note removed: "I3C voltage level translation"
- note removed: "Pull up via 10KOhm"
- note removed: "USB CLIENT"
- note removed: "USB HOST"
- note removed: "reserved for future use (as of DC-SCI OPC specification)"
- moved on the sheet: C107, C135, C139, C149, C154, C162, C166, C168, C169, C170, C172, C173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
